File: Eagle/MazeSolverPCB_v_0.2_.brd (EAGLE design)
At the start: 53.3 x 47.9 mm, 26 parts

Commit message: Updated PCB
Routing:
- net N$1: track 0.00 -> 167.8 mm
- net N$2: track 0.00 -> 67.8 mm
- net N$21: track 0.00 -> 52.4 mm
- net N$20: track 0.00 -> 48.3 mm
- net N$12: track 0.00 -> 44.5 mm
- net N$26: track 0.00 -> 44.0 mm
- net N$13: track 0.00 -> 42.7 mm
- net N$10: track 0.00 -> 34.8 mm
- net N$27: track 0.00 -> 32.9 mm
- net N$3: track 0.00 -> 30.7 mm
- net N$15: track 0.00 -> 30.3 mm
- net N$24: track 0.00 -> 24.8 mm
- net N$14: track 0.00 -> 22.3 mm
- net N$30: track 0.00 -> 16.9 mm
- net N$28: track 0.00 -> 15.7 mm
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Other:
- board size 53.3 x 47.9 mm -> 53.3 x 50.8 mm
